Commit message: Add files via upload

File: articubot_one/description/robot_core.xacro (robot description, xacro)
@@ -9,10 +9,10 @@
     <xacro:property name="wheel_thickness" value="0.050"/>
     <xacro:property name="wheel_mass" value="0.05"/>
-    <xacro:property name="wheel_offset_x" value="0.280"/>
+    <xacro:property name="wheel_offset_x" value="0.075"/>
     <xacro:property name="wheel_offset_y" value="0.230"/>
     <xacro:property name="wheel_offset_z" value="0.050"/>
     <xacro:property name="caster_wheel_radius" value="0.05"/>
-    <xacro:property name="caster_wheel_mass" value="0.01"/>
-    <xacro:property name="caster_wheel_offset_x" value="0.075"/>
+    <xacro:property name="caster_wheel_mass" value="0.1"/>
+    <xacro:property name="caster_wheel_offset_x" value="0.280"/>
     <xacro:property name="caster_wheel_offset_z" value="${wheel_offset_z - wheel_radius + caster_wheel_radius}"/>
     <material name="white">
